Commit message: fix camera static

File: catkin_ws/src/scene/urdf/camera.urdf (robot description, URDF)
Before this commit: robot camera, 1 links, 0 joints
Links:
- link camera_link: mass 1 -> 0.01

File: catkin_ws/src/scene/urdf/puck.urdf (robot description, URDF)
Before this commit: robot puck, 1 links, 0 joints
Links:
- link puck_link: mass 0.15 -> 0.1
