Commit message: merge camera, plane and borders in URDF

File: catkin_ws/src/scene/urdf/table.urdf (robot description, URDF)
Before this commit: robot table, 1 links, 0 joints
Links:
- added link table_borders_link, mass 10.0; collision mesh filename=package://scene/models/table_borders/meshes/airhockey-borde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 scale=0.001 0.001 0.001; visual mesh filename=package://scene/models/table_borders/meshes/airhockey-borde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 scale=0.001 0.001 0.001
- link table_link: geometry collision mesh filename=package://scene/models/plane/meshes/airhockey-plane.stl scale=0.001 0.001 0.001; visual mesh filename=package://scene/models/plane/meshes/airhockey-plane.dae scale=0.001 0.001 0.001
Joints:
- added joint table_fixed: type fixed, parent table_link, child table_borders_link, origin xyz=0 0 0
