Commit message: modified move_franka

File: catkin_ws/src/end_effector/urdfs/robot_compose.urdf.xacro (robot description, xacro)
@@ -6,5 +6,5 @@
         <parent link="panda_link8"/>
         <child link="stick_link"/>
-        <origin xyz="0 0 0.4" rpy="0 0 0"/>
+        <origin xyz="0 0 0.8" rpy="0 0 0"/>
     </joint>
 </robot>

File: catkin_ws/src/franka_ros/franka_description/robots/common/franka_arm.xacro (robot description, xacro)
@@ -90,5 +90,5 @@
     </xacro:link_with_sc>
     <joint name="${arm_id}_joint6" type="revolute">
-      <origin rpy="${pi/2} ${-pi/2} 0" xyz="0 0 0" />
+      <origin rpy="${pi/2} 0 0" xyz="0 0 0" />
       <parent link="${arm_id}_link5" />
       <child link="${arm_id}_link6" />

Commit message: modifications to move_franka

File: catkin_ws/src/end_effector/urdfs/robot_compose.urdf.xacro (robot description, xacro)
@@ -6,5 +6,5 @@
         <parent link="panda_link8"/>
         <child link="stick_link"/>
-        <origin xyz="0 0 0.8" rpy="0 0 0"/>
+        <origin xyz="0 0 0.4" rpy="0 0 0"/>
     </joint>
 </robot>
