Commit message: move_franka corrections to frames orientation and position

File: catkin_ws/src/end_effector/urdfs/ef.urdf (robot description, URDF)
Before this commit: robot end_effector, 7 links, 6 joints
Links:
- added link ef_start
Joints:
- added joint start_stick_joint: type fixed, parent ef_start, child stick_link, origin xyz=0 0 0 rpy=0 3.9268 0
- joint stick_tmp0_joint: origin xyz=0 0 -0.21 rpy=0 -0.7853 0 -> xyz=0 0 -0.21 rpy=0 0.7853 3.1415

File: catkin_ws/src/end_effector/urdfs/robot_compose.urdf.xacro (robot description, xacro)
@@ -5,6 +5,6 @@
     <joint name="rbt_ef_joint" type="fixed">
         <parent link="panda_link8"/>
-        <child link="stick_link"/>
-        <origin xyz="0 0 0" rpy="0 3.9268 0"/>
+        <child link="ef_start"/>
+        <origin xyz="0 0 0" rpy="0 0 0"/>
     </joint>
 </robot>

Commit message: Add prof tool
Change from our tool to prof tool

File: catkin_ws/src/end_effector/urdfs/ef.urdf (robot description, URDF)
Before this commit: robot end_effector, 8 links, 7 joints
Links:
- removed link ef_start
- link paddle_link: geometry visual mesh filename=package://end_effector/models/AD_Piattello-Snodo_Assieme.stl scale=0.001 0.001 0.001
- link spring_link: geometry 
- link stick_link: geometry visual mesh filename=package://end_effector/models/AD_Flangia-Asta_Assieme.stl scale=0.001 0.001 0.001
Joints:
- removed joint start_stick_joint
- joint spring_paddle_joint: origin xyz=0.0 0.0 -0.06 rpy=0 0 0 -> xyz=0.0 0.0 0 rpy=0 -0.7853 0
- joint stick_tmp0_joint: origin xyz=0 0 -0.21 rpy=0 0.7853 3.1415 -> xyz=0 0 0 rpy=0 0 0
- joint tmp2_tmp3_joint: origin xyz=0 0 0 rpy=0 -0.7853 0 -> xyz=0 0 0 rpy=0 0 0

File: catkin_ws/src/end_effector/urdfs/robot_compose.urdf.xacro (robot description, xacro)
@@ -5,6 +5,6 @@
     <joint name="rbt_ef_joint" type="fixed">
         <parent link="panda_link8"/>
-        <child link="ef_start"/>
-        <origin xyz="0 0 0" rpy="0 0 0"/>
+        <child link="stick_link"/>
+        <origin xyz="0 0 0.595" rpy="0 0 0"/>
     </joint>
 </robot>

Commit message: prof end_effector

File: catkin_ws/src/end_effector/urdfs/ef.urdf (robot description, URDF)
Before this commit: robot end_effector, 7 links, 6 joints
Links:
- link paddle_link: geometry visual mesh filename=package://end_effector/models/mallet.stl scale=1 1 1
- link stick_link: geometry visual mesh filename=package://end_effector/models/stick.stl scale=1 1 1
Joints:
- joint spring_paddle_joint: origin xyz=0.0 0.0 0 rpy=0 -0.7853 0 -> xyz=0.0 0.0 0.0 rpy=0 ${pi/4} 0

File: catkin_ws/src/end_effector/urdfs/robot_compose.urdf.xacro (robot description, xacro)
@@ -6,5 +6,5 @@
         <parent link="panda_link8"/>
         <child link="stick_link"/>
-        <origin xyz="0 0 0.595" rpy="0 0 0"/>
+        <origin xyz="0 0 ${0.4+0.03}" rpy="0 0 0"/>
     </joint>
 </robot>

File: catkin_ws/src/franka_ros/franka_description/robots/common/franka_arm.xacro (robot description, xacro)
@@ -90,5 +90,5 @@
     </xacro:link_with_sc>
     <joint name="${arm_id}_joint6" type="revolute">
-      <origin rpy="${pi/2} 0 0" xyz="0 0 0" />
+      <origin rpy="${pi/2} ${-pi/2} 0" xyz="0 0 0" />
       <parent link="${arm_id}_link5" />
       <child link="${arm_id}_link6" />

Commit message: simplified end_effector

File: catkin_ws/src/end_effector/urdfs/ef.urdf (robot description, URDF)
Before this commit: robot end_effector, 7 links, 6 joints
Links:
- link paddle_link: geometry collision mesh filename=package://end_effector/models/mallet.stl scale=0.001 0.001 0.001; visual mesh filename=package://end_effector/models/mallet.stl scale=0.001 0.001 0.001
- link stick_link: geometry visual mesh filename=package://end_effector/models/stick.stl scale=0.001 0.001 0.001
Joints:
- joint spring_paddle_joint: origin xyz=0.0 0.0 0.0 rpy=0 ${pi/4} 0 -> xyz=0 0 0 rpy=0 ${3*pi/4} 0

File: catkin_ws/src/end_effector/urdfs/robot_compose.urdf.xacro (robot description, xacro)
@@ -6,5 +6,5 @@
         <parent link="panda_link8"/>
         <child link="stick_link"/>
-        <origin xyz="0 0 ${0.4+0.03}" rpy="0 0 0"/>
+        <origin xyz="0 0 0.4" rpy="0 0 0"/>
     </joint>
 </robot>

Commit message: end_effector modification

File: catkin_ws/src/end_effector/urdfs/ef.urdf (robot description, URDF)
Before this commit: robot end_effector, 7 links, 6 joints
Links:
- removed link paddle_link
- removed link spring_link
- removed link tmp0
- removed link tmp1
- removed link tmp2
- removed link tmp3
- added link mallet_link, mass 0.1; visual mesh filename=package://end_effector/models/mallet.stl scale=0.001 0.001 0.001
- added link tmp_link, mass 0.1
Joints:
- removed joint spring_paddle_joint
- removed joint stick_tmp0_joint
- removed joint tmp0_tmp1_joint
- removed joint tmp1_tmp2_joint
- removed joint tmp2_tmp3_joint
- removed joint tmp3_spring_joint
- added joint stick_tmp_joint: type fixed, parent stick_link, child tmp_link, origin xyz=0 0 0 rpy=0 ${-pi/6} 0
- added joint tmp_mallet_joint: type fixed, parent tmp_link, child mallet_link, origin xyz=0 0 0.12 rpy=0 0 0

Commit message: cartesian_path movement

File: catkin_ws/src/end_effector/urdfs/ef.urdf (robot description, URDF)
Before this commit: robot end_effector, 3 links, 2 joints
Joints:
- joint stick_tmp_joint: origin xyz=0 0 0 rpy=0 ${-pi/6} 0 -> xyz=0 0 0 rpy=0 ${-pi/3} 0
- joint tmp_mallet_joint: origin xyz=0 0 0.12 rpy=0 0 0 -> xyz=0 0 0.1 rpy=0 0 0

Commit message: move_franka finished

File: catkin_ws/src/end_effector/urdfs/ef.urdf (robot description, URDF)
Before this commit: robot end_effector, 3 links, 2 joints
Joints:
- joint stick_tmp_joint: origin xyz=0 0 0 rpy=0 ${-pi/3} 0 -> xyz=0 0 0 rpy=0 ${-pi/4} 0

Commit message: Code with Movit motion completed

File: catkin_ws/src/end_effector/urdfs/ef.urdf (robot description, URDF)
Before this commit: robot end_effector, 3 links, 2 joints
Links:
- link mallet_link: mass 0.1 -> 0.5
